File: PCB/hidroboat_pcb/hidroboat_pcb.kicad_sch (KiCad schematic)
At the start: 10 parts, among them J1 RTCLOCK, J2 SDCARD, J3 GPS, J4 DHT11, J5 RELE 5V, U1 Heltec_Wifi_LoRa_V1, U2 YAAJ_DCDC_StepDown_LM2596, U3 L7805

Commit message: att esquematico
rotulos, ligações
Parts:
- removed C1, C2: 3.3uf, Capacitor_THT:C_Radial_D5.0mm_H11.0mm_P2.00mm, symbol Device:C
- removed U3: L7805, l7805:TO255P1020X450X2000-3, symbol Regulator_Linear:L7805
- added J1, J11, J12, J13, J15, J17, J4, J5, J7, J8, J9: Conn_02x01, symbol Connector_Generic:Conn_02x01
- added J18: Conn_01x02, Connector_Phoenix_MC_HighVoltage:PhoenixContact_MCV_1,5_2-G-5.08_1x02_P5.08mm_Vertical, symbol Connector_Generic:Conn_01x02
- added J19, J20, J21, J22, J23, J24: Conn_01x06_Socket, Connector_PinSocket_2.54mm:PinSocket_1x06_P2.54mm_Vertical, symbol Connector:Conn_01x06_Socket
- added J3: TempAgua, symbol Connector_Generic:Conn_01x03
- added R1, R2, R3: 4.7K, symbol Device:R
- renumbered J1 to J10, J5 to J14, J3 to J16, J4 to J2, J2 to J6
Connections:
- net VCC is gone; now on net +5V: U2.4 (Vout)
- net +12V: now also J18.1 (Pin_1), J19.1 (Pin_1), J19.2 (Pin_2), J19.3 (Pin_3), J19.4 (Pin_4), J19.5 (Pin_5), J19.6 (Pin_6)
- net +5V: now also J14.2 (5v), J6.2 (Pin_2), U1.2 (5V), J20.1 (Pin_1), J20.2 (Pin_2), J20.3 (Pin_3), J20.4 (Pin_4), J20.5 (Pin_5), J20.6 (Pin_6)
- net GND: now also J10.5 (GND), J14.3 (GND), J16.1 (GND), J2.4 (GND), J6.1 (Pin_1), U1.1 (GND), J23.1 (Pin_1), J23.2 (Pin_2), J23.3 (Pin_3), J23.4 (Pin_4), J23.5 (Pin_5), J23.6 (Pin_6), J24.1 (Pin_1), J24.2 (Pin_2), J24.3 (Pin_3), J24.4 (Pin_4), J24.5 (Pin_5), J24.6 (Pin_6), J3.2 (GND); no longer U2.2 (GND)
- net at J10.3 (SCL): now also J9.2 (Pin_2), R2.2
- net at J10.4 (SDA): now also J12.2 (Pin_2), R1.2
- net +3.3V: now reaches J10.6 (VCC)
- net +3.3V: now also J16.4 (VCC), J2.1 (3.3V), J2.2 (GPIO21), U1.34 (3V3), J1.2 (Pin_2), J21.1 (Pin_1), J21.2 (Pin_2), J21.3 (Pin_3), J21.4 (Pin_4), J21.5 (Pin_5), J21.6 (Pin_6), J3.1 (3.3v), R1.1, R2.1, R3.2
- net at J6.3 (Pin_3): now also J5.2 (Pin_2)
- net at J6.4 (Pin_4): now also J7.2 (Pin_2)
- net at J6.5 (Pin_5): now also J8.2 (Pin_2)
- net at J6.6 (Pin_6): now also J11.2 (Pin_2)
- net at J14.1 (Signal): now also J13.2 (Pin_2)
- net at J16.2 (TX): now also J17.2 (Pin_2)
- net at J16.3 (RX): now also J15.2 (Pin_2)
- net GPIO23: now reaches U1.11 (V_SPI_D/GPIO23)
- net GPIO23: now also J11.1 (Pin_1)
- net GPIO15: now reaches U1.14 (OLED_SCL/TOUCH3/HSPI_CS0/ADC2_3/GPIO15)
- net GPIO15: now also J9.1 (Pin_1)
- net GPIO2: now reaches U1.15 (TOUCH2/HSPI_WP/ADC2_2/GPIO2)
- net GPIO2: now also J4.1 (Pin_1)
- net GPIO4: now reaches U1.16 (OLED_SDA/TOUCH0/HSPI_HD/ADC2_0/GPIO4)
- net GPIO4: now also J12.1 (Pin_1)
- net GPIO17: now reaches U1.17 (U2_TX/GPIO17)
- net GPIO17: now also J8.1 (Pin_1)
- net GPIO21: now reaches U1.19 (V_SPI_HD/SDA/GPIO21)
- net GPIO21: now also J1.1 (Pin_1)
- net GPIO13: now reaches U1.20 (TOUCH4/ADC2_4/GPIO13)
- net GPIO13: now also J5.1 (Pin_1)
- net GPIO12: now reaches U1.21 (TOUCH5/ADC2_5/GPIO12)
- net GPIO12: now also J7.1 (Pin_1)
- net GPIO25: now reaches U1.25 (LED/DAC2/ADC2_8/GPIO25)
- net GPIO25: now also J13.1 (Pin_1)
- net TX: now reaches U1.5 (U0_RX/GPIO3)
- net TX: now also J17.1 (Pin_1)
- net RX: now reaches U1.6 (U0_TX/GPIO1)
- net RX: now also J15.1 (Pin_1)
- new net: J3.3 (GPIO2), J4.2 (Pin_2), R3.1
- new net GNDREF: J18.2 (Pin_2), J22.1 (Pin_1), J22.2 (Pin_2), J22.3 (Pin_3), J22.4 (Pin_4), J22.5 (Pin_5), J22.6 (Pin_6), U2.2 (GND)
- no-connect marks 0 -> 25
Other:
- moved on the sheet: J10, J14, J16, J2, J6, U1, U2

Commit message: add footprint
Parts:
- added F1: Fuse_Small, Fuse:Fuse_Blade_Mini_directSolder, symbol Device:Fuse_Small
- added J31: Conn_01x15, Connector_PinSocket_2.54mm:PinSocket_1x15_P2.54mm_Vertical, symbol Connector_Generic:Conn_01x15
- added J7: Conn_01x14, Connector_PinSocket_2.54mm:PinSocket_1x14_P2.54mm_Vertical, symbol Connector_Generic:Conn_01x14
- added R1: 4.7K, Resistor_THT:R_Axial_DIN0207_L6.3mm_D2.5mm_P7.62mm_Horizontal, symbol Device:R
- J1: footprint (none) -> Connector_PinHeader_2.54mm:PinHeader_1x03_P2.54mm_Vertical
- J10: renamed from J5; footprint (none) -> Connector_PinHeader_2.54mm:PinHeader_1x03_P2.54mm_Vertical
- J11: renamed from J7; footprint (none) -> Connector_PinHeader_2.54mm:PinHeader_1x03_P2.54mm_Vertical
- J12: renamed from J8; footprint (none) -> Connector_PinHeader_2.54mm:PinHeader_1x03_P2.54mm_Vertical
- J13: renamed from J11; footprint (none) -> Connector_PinHeader_2.54mm:PinHeader_1x03_P2.54mm_Vertical
- J15: renamed from J20; footprint Connector_PinSocket_2.54mm:PinSocket_1x06_P2.54mm_Vertical -> Connector_PinSocket_2.54mm:PinSocket_2x03_P2.54mm_Vertical
- J16: renamed from J23; footprint Connector_PinSocket_2.54mm:PinSocket_1x06_P2.54mm_Vertical -> Connector_PinSocket_2.54mm:PinSocket_2x03_P2.54mm_Vertical
- J17: renamed from J21; footprint Connector_PinSocket_2.54mm:PinSocket_1x06_P2.54mm_Vertical -> Connector_PinSocket_2.54mm:PinSocket_2x03_P2.54mm_Vertical
- J18: renamed from J24; footprint Connector_PinSocket_2.54mm:PinSocket_1x06_P2.54mm_Vertical -> Connector_PinSocket_2.54mm:PinSocket_2x03_P2.54mm_Vertical
- J26: renamed from J4; footprint (none) -> Connector_PinHeader_2.54mm:PinHeader_1x03_P2.54mm_Vertical
- J27: renamed from J3; footprint (none) -> Connector_PinSocket_2.54mm:PinSocket_1x03_P2.54mm_Vertical
- J28: renamed from J9; footprint (none) -> Connector_PinHeader_2.54mm:PinHeader_1x03_P2.54mm_Vertical
- J29: renamed from J12; footprint (none) -> Connector_PinHeader_2.54mm:PinHeader_1x03_P2.54mm_Vertical
- J3: renamed from J18; footprint Connector_Phoenix_MC_HighVoltage:PhoenixContact_MCV_1,5_2-G-5.08_1x02_P5.08mm_Vertical -> Connector_PinSocket_2.54mm:PinSocket_1x02_P2.54mm_Vertical
- J30: renamed from J13; footprint (none) -> Connector_PinHeader_2.54mm:PinHeader_1x03_P2.54mm_Vertical
- J5: renamed from J15; footprint (none) -> Connector_PinHeader_2.54mm:PinHeader_1x03_P2.54mm_Vertical
- J6: renamed from J17; footprint (none) -> Connector_PinHeader_2.54mm:PinHeader_1x03_P2.54mm_Vertical
- J8: renamed from J19; footprint Connector_PinSocket_2.54mm:PinSocket_1x06_P2.54mm_Vertical -> Connector_PinSocket_2.54mm:PinSocket_2x03_P2.54mm_Vertical
- J9: renamed from J22; footprint Connector_PinSocket_2.54mm:PinSocket_1x06_P2.54mm_Vertical -> Connector_PinSocket_2.54mm:PinSocket_2x03_P2.54mm_Vertical
- R2: renamed from R3; footprint (none) -> Resistor_THT:R_Axial_DIN0207_L6.3mm_D2.5mm_P7.62mm_Horizontal
- R3: renamed from R1; footprint (none) -> Resistor_THT:R_Axial_DIN0207_L6.3mm_D2.5mm_P7.62mm_Horizontal
- R4: renamed from R2; footprint (none) -> Resistor_THT:R_Axial_DIN0207_L6.3mm_D2.5mm_P7.62mm_Horizontal
- renumbered J6 to J14, J16 to J2, J14 to J32, J10 to J33, J2 to J4, U2 to U1, U1 to U2
Connections:
- net +12V: now also F1.1; no longer U1.1 (Vin)
- net +3.3V: now also R1.2; no longer J1.2 (Pin_2), J4.2 (GPIO21)
- net GPIO12: now also J31.13 (Pin_13)
- net GPIO13: now also J31.14 (Pin_14)
- net GPIO15: now also J7.5 (Pin_5)
- net GPIO17: now also J7.2 (Pin_2)
- net GPIO2: now also J7.4 (Pin_4)
- net GPIO21: now also J31.15 (Pin_15)
- net GPIO23: now also J7.8 (Pin_8)
- net GPIO25: now also J31.9 (Pin_9)
- net GPIO4: now also J7.3 (Pin_3)
- net RX: now also J7.13 (Pin_13)
- net TX: now also J7.14 (Pin_14)
- net GPIO19: now reaches U2.10 (LORA_MISO/U0_CTS/V_SPI_Q/GPIO19)
- net GPIO19: now also J7.9 (Pin_9)
- net GPIO18: now reaches U2.12 (LORA_CS/V_SPI_CLK/GPIO18)
- net GPIO18: now also J7.7 (Pin_7)
- net GPIO5: now reaches U2.13 (LORA_SCK/V_SPI_CS0/GPIO5)
- net GPIO5: now also J7.6 (Pin_6)
- net GPIO16: now reaches U2.18 (OLED_RST/U2_RX/GPIO16)
- net GPIO16: now also J7.1 (Pin_1)
- net GPIO14: now reaches U2.22 (LORA_RST/TOUCH6/ADC2_6/GPIO14)
- net GPIO14: now also J31.12 (Pin_12)
- net GPIO27: now reaches U2.23 (LORA_MOSI/TOUCH7/ADC2_7/GPIO27)
- net GPIO27: now also J31.11 (Pin_11)
- net GPIO26: now reaches U2.24 (LORA_DIO0/DAC1/ADC2_9/GPIO26)
- net GPIO26: now also J31.10 (Pin_10)
- net GPIO33: now reaches U2.26 (LORA_DIO1/XTAL32/TOUCH8/ADC1_5/GPIO33)
- net GPIO33: now also J31.8 (Pin_8)
- net GPIO32: now reaches U2.27 (LORA_DIO2/XTAL32/TOUCH9/ADC1_4/GPIO32)
- net GPIO32: now also J31.7 (Pin_7)
- net GPIO35: now reaches U2.28 (ADC1_7/GPIO35)
- net GPIO35: now also J31.6 (Pin_6)
- net GPIO34: now reaches U2.29 (ADC1_6/GPIO34)
- net GPIO34: now also J31.5 (Pin_5)
- net GPIO39: now reaches U2.30 (ADC1_3/GPIO39)
- net GPIO39: now also J31.4 (Pin_4)
- net GPIO38: now reaches U2.31 (ADC1_2/GPIO38)
- net GPIO38: now also J31.3 (Pin_3)
- net GPIO37: now reaches U2.32 (ADC1_1/GPIO37)
- net GPIO37: now also J31.2 (Pin_2)
- net GPIO36: now reaches U2.33 (ADC1_0/GPIO36)
- net GPIO36: now also J31.1 (Pin_1)
- net RST: now reaches U2.7 (RST)
- net RST: now also J7.12 (Pin_12)
- net GPIO0: now reaches U2.8 (PRG_BUTTON/TOUCH1/ADC2_1/GPIO0)
- net GPIO0: now also J7.11 (Pin_11)
- net GPIO22: now reaches U2.9 (U0_RTS/V_SPI_WP/SCL/GPIO22)
- net GPIO22: now also J7.10 (Pin_10)
- new net: J1.2 (Pin_2), J4.2 (Pin_2), R1.1
- new net: F1.2, U1.1 (Vin)
- no-connect marks 25 -> 7
Other:
- moved on the sheet: J14, J15, J16, J2, J30, J32, J33, J5, J6
